File: VGA_PANEL_BREAKOUT.kicad_pcb (KiCad board)
At the start: 2 copper layers, 15 x 20.5 mm, 32 parts, among them J1 DB15_Female_HighDensity

Commit message: Initial commit
Parts:
- removed the REF** at (164.1, 109.0)
- removed the REF** at (157.2, 109.0)
- removed the REF** at (166.3, 109.0)
- turned J1 to 180 degrees
Connections:
- REF** pad 1: (no net) -> VSYNC
- REF** pad 1: GND -> RED
- REF** pad 1: VSYNC -> GREEN
- REF** pad 1: HSYNC -> BLUE
- REF** pad 1: BLUE -> HSYNC
- REF** pad 1: GREEN -> VSYNC
- REF** pad 1: RED -> GND
- REF** pad 1: BLUE -> RED (x2)
- REF** pad 1: RED -> BLUE (x2)
Routing:
- net GND: track 27.7 -> 38.3 mm
- net GREEN: track 22.9 -> 28.5 mm
- net RED: track 16.8 -> 21.5 mm, vias 1 -> 2
- net HSYNC: track 6.94 -> 6.13 mm
- net BLUE: track 24.1 -> 23.8 mm, vias 2 -> 1
Other:
- board text added: "R G B H V"
- board text removed: "V H B G R"

Commit message: Initial Commit
First working design.
Routing:
- net GND: track 38.3 -> 37.7 mm
Other:
- board text added: "Licensed under CERN-OHL-S v2"
Changed lines of the file:
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@@
   (general
     (thickness 1.6)
-    (drawings 24)
-    (tracks 85)
+    (drawings 25)
+    (tracks 90)
     (zones 0)
     (modules 29)
@@
   )
   (page A4)
+  (title_block
+    (title "VGA Panel Breakout")
+    (date 2020-06-27)
+    (company Tinkerplunk)
+    (comment 1 "Copyright Tinkerplunk 2020. Licensed under CERN-OHL-S v2")
+  )
   (layers
     (0 F.Cu signal)
@@
     (visible_elements 7FFFFFFF)
     (pcbplotparams
-      (layerselection 0x010fc_ffffffff)
+      (layerselection 0x010f0_ffffffff)
       (usegerberextensions true)
       (usegerberattributes false)
@@
     (pad "" np_thru_hole circle (at 0 0) (size 0.3 0.3) (drill 0.3) (layers *.Cu *.Mask))
   )
+  (gr_text "Licensed under\nCERN-OHL-S v2" (at 161.7 103.5) (layer B.SilkS)
+    (effects (font (size 1 1) (thickness 0.15)) (justify mirror))
+  )
   (gr_text GND (at 155.8 96 180) (layer F.SilkS)
     (effects (font (size 0.6 0.6) (thickness 0.15)))
@@
   (segment (start 158.549999 95.250001) (end 159.248997 95.250001) (width 0.25) (layer B.Cu) (net 1))
   (segment (start 157.8 96) (end 158.549999 95.250001) (width 0.25) (layer B.Cu) (net 1))
-  (segment (start 167.225001 107.574999) (end 167.225001 105.751999) (width 0.25) (layer B.Cu) (net 1))
-  (segment (start 166.5 109.05) (end 166.5 108.3) (width 0.25) (layer B.Cu) (net 1))
-  (segment (start 167.225001 105.751999) (end 165.973002 104.5) (width 0.25) (layer B.Cu) (net 1))
-  (segment (start 166.5 108.3) (end 167.225001 107.574999) (width 0.25) (layer B.Cu) (net 1))
   (via (at 156.712347 105.812347) (size 0.8) (drill 0.4) (layers F.Cu B.Cu) (net 1))
-  (segment (start 165.973002 104.5) (end 158.024694 104.5) (width 0.25) (layer B.Cu) (net 1))
-  (segment (start 158.024694 104.5) (end 156.712347 105.812347) (width 0.25) (layer B.Cu) (net 1))
   (segment (start 155.25 105.3) (end 155.25 103.55) (width 0.25) (layer F.Cu) (net 1))
   (segment (start 155.762347 105.812347) (end 155.25 105.3) (width 0.25) (layer F.Cu) (net 1))
   (segment (start 156.712347 105.812347) (end 155.762347 105.812347) (width 0.25) (layer F.Cu) (net 1))
+  (segment (start 157.324694 105.2) (end 156.712347 105.812347) (width 0.25) (layer B.Cu) (net 1))
+  (segment (start 166.673002 105.2) (end 157.324694 105.2) (width 0.25) (layer B.Cu) (net 1))
+  (segment (start 167.225001 107.574999) (end 167.225001 105.751999) (width 0.25) (layer B.Cu) (net 1))
+  (segment (start 166.5 109.05) (end 166.5 108.3) (width 0.25) (layer B.Cu) (net 1))
+  (segment (start 166.5 108.3) (end 167.225001 107.574999) (width 0.25) (layer B.Cu) (net 1))
+  (segment (start 167.225001 105.751999) (end 166.673002 105.2) (width 0.25) (layer B.Cu) (net 1))
   (segment (start 166.87566 97.98) (end 168.4 96.45566) (width 0.25) (layer B.Cu) (net 2))
   (segment (start 165.815 97.98) (end 166.87566 97.98) (width 0.25) (layer B.Cu) (net 2))
@@
   (segment (start 165.25 104.65) (end 165.25 103.55) (width 0.25) (layer F.Cu) (net 3))
   (segment (start 163.9 106) (end 165.25 104.65) (width 0.25) (layer F.Cu) (net 3))
-  (segment (start 160.2 106.6) (end 163.3 106.6) (width 0.25) (layer B.Cu) (net 3))
-  (segment (start 163.3 106.6) (end 163.9 106) (width 0.25) (layer B.Cu) (net 3))
+  (segment (start 163.500001 106.399999) (end 163.9 106) (width 0.25) (layer B.Cu) (net 3))
+  (segment (start 163.249989 106.650011) (end 163.500001 106.399999) (width 0.25) (layer B.Cu) (net 3))
+  (segment (start 160 106.8) (end 160.149989 106.650011) (width 0.25) (layer B.Cu) (net 3))
   (segment (start 160 109.05) (end 160 106.8) (width 0.25) (layer B.Cu) (net 3))
-  (segment (start 160 106.8) (end 160.2 106.6) (width 0.25) (layer B.Cu) (net 3))
+  (segment (start 160.149989 106.650011) (end 163.249989 106.650011) (width 0.25) (layer B.Cu) (net 3))
   (segment (start 155.975013 95.095001) (end 154.64999 93.769978) (width 0.25) (layer F.Cu) (net 4))
   (segment (start 154.64999 93.769978) (end 154.64999 91.80001) (width 0.25) (layer F.Cu) (net 4))
@@
   (segment (start 157.171001 95.095001) (end 155.975013 95.095001) (width 0.25) (layer F.Cu) (net 4))
   (segment (start 161.235 97.98) (end 160.485001 97.230001) (width 0.25) (layer F.Cu) (net 4))
+  (segment (start 162.75 103.55) (end 162.75 105.3) (width 0.25) (layer F.Cu) (net 4))
+  (segment (start 156.75 106.8) (end 157.695153 105.854847) (width 0.25) (layer B.Cu) (net 4))
+  (segment (start 162.75 105.3) (end 162.12499 105.92501) (width 0.25) (layer F.Cu) (net 4))
+  (segment (start 161.279468 105.92501) (end 161.845153 105.92501) (width 0.25) (layer B.Cu) (net 4))
+  (segment (start 161.209305 105.854847) (end 161.279468 105.92501) (width 0.25) (layer B.Cu) (net 4))
   (segment (start 156.75 109.05) (end 156.75 106.8) (width 0.25) (layer B.Cu) (net 4))
-  (via (at 161.845153 105.854847) (size 0.8) (drill 0.4) (layers F.Cu B.Cu) (net 4))
-  (segment (start 157.695153 105.854847) (end 161.845153 105.854847) (width 0.25) (layer B.Cu) (net 4))
-  (segment (start 156.75 106.8) (end 157.695153 105.854847) (width 0.25) (layer B.Cu) (net 4))
-  (segment (start 162.75 104.95) (end 162.75 103.55) (width 0.25) (layer F.Cu) (net 4))
-  (segment (start 161.845153 105.854847) (end 162.75 104.95) (width 0.25) (layer F.Cu) (net 4))
-  (segment (start 161.765 109.05) (end 161.765 106.8) (width 0.25) (layer F.Cu) (net 9))
-  (segment (start 160.25 105.285) (end 160.25 103.55) (width 0.25) (layer F.Cu) (net 9))
-  (segment (start 161.765 106.8) (end 160.25 105.285) (width 0.25) (layer F.Cu) (net 9))
+  (segment (start 157.695153 105.854847) (end 161.209305 105.854847) (width 0.25) (layer B.Cu) (net 4))
+  (via (at 161.845153 105.92501) (size 0.8) (drill 0.4) (layers F.Cu B.Cu) (net 4))
+  (segment (start 162.12499 105.92501) (end 161.845153 105.92501) (width 0.25) (layer F.Cu) (net 4))
+  (segment (start 160.25 106.285) (end 160.25 105.3) (width 0.25) (layer F.Cu) (net 9))
+  (segment (start 160.25 105.3) (end 160.25 103.55) (width 0.25) (layer F.Cu) (net 9))
+  (segment (start 161.765 109.05) (end 161.765 107.8) (width 0.25) (layer F.Cu) (net 9))
+  (segment (start 161.765 107.8) (end 160.25 106.285) (width 0.25) (layer F.Cu) (net 9))
   (segment (start 159.475 109.075) (end 159.475 109.05) (width 0.25) (layer F.Cu) (net 10))
   (segment (start 157.75 105.075) (end 157.75 103.55) (width 0.25) (layer F.Cu) (net 10))
